Commit message: Automatic update of urdf triggered by GitHub Action
r1-models = c449502905b980ad6bcc30b86da93efbfad48a21
cad-libraries    = https://github.com/icub-tech-iit/cad-libraries/commit/afe728d39d327621ffae7325d3ef17c46c503bf1
cad-mechanics    = https://github.com/icub-tech-iit/cad-mechanics/commit/ce2cb436e4400628e829bbfa0f29caf4592700df
creo2urdf        = https://github.com/icub-tech-iit/creo2urdf/releases/tag/v0.5.18

File: urdf/R1Mk3/robots/R1Mk3Gazebo/model.urdf (robot description, URDF)
Before this commit: robot R1Mk3, 184 links, 183 joints
Joints:
- joint depth_fixed_joint: origin xyz=0.05132675386498539 0.04448710000000006 0.05375475275483321 rpy=-1.3962634015954642 -1.0632884247878182e-17 -1.5707963267948954 -> xyz=0.05132675386498539 0.04448710000000006 0.05375475275483321 rpy=3.6174008641979e-6 3.4015943103992236e-6 6.378576785263269e-7
- joint depth_rgb_fixed_joint: origin xyz=0.05132675386498542 0.01848710000000006 0.05375475275483321 rpy=-1.3962634015954642 -1.0632884247878182e-17 -1.5707963267948954 -> xyz=0.05132675386498542 0.01848710000000006 0.05375475275483321 rpy=3.6174008641979e-6 3.4015943103992236e-6 6.378576785263269e-7

File: urdf/R1Mk3/robots/R1Mk3Gazebo_minContacts/model.urdf (robot description, URDF)
Before this commit: robot R1Mk3, 184 links, 183 joints
Joints:
- joint depth_fixed_joint: origin xyz=0.05132675386498539 0.04448710000000006 0.05375475275483321 rpy=-1.3962634015954642 -1.0632884247878182e-17 -1.5707963267948954 -> xyz=0.05132675386498539 0.04448710000000006 0.05375475275483321 rpy=3.6174008641979e-6 3.4015943103992236e-6 6.378576785263269e-7
- joint depth_rgb_fixed_joint: origin xyz=0.05132675386498542 0.01848710000000006 0.05375475275483321 rpy=-1.3962634015954642 -1.0632884247878182e-17 -1.5707963267948954 -> xyz=0.05132675386498542 0.01848710000000006 0.05375475275483321 rpy=3.6174008641979e-6 3.4015943103992236e-6 6.378576785263269e-7

File: urdf/R1Mk3/robots/R1SN003/model.urdf (robot description, URDF)
Before this commit: robot R1Mk3, 184 links, 183 joints
Joints:
- joint depth_fixed_joint: origin xyz=0.05132675386498539 0.04448710000000006 0.05375475275483321 rpy=-1.3962634015954642 -1.0632884247878182e-17 -1.5707963267948954 -> xyz=0.05132675386498539 0.04448710000000006 0.05375475275483321 rpy=3.6174008641979e-6 3.4015943103992236e-6 6.378576785263269e-7
- joint depth_rgb_fixed_joint: origin xyz=0.05132675386498542 0.01848710000000006 0.05375475275483321 rpy=-1.3962634015954642 -1.0632884247878182e-17 -1.5707963267948954 -> xyz=0.05132675386498542 0.01848710000000006 0.05375475275483321 rpy=3.6174008641979e-6 3.4015943103992236e-6 6.378576785263269e-7
