Commit message: urdf

File: urdf/R1Mk3/robots/R1Mk3Gazebo_minContacts/model.urdf (robot description, URDF)
Before this commit: robot R1Mk3, 184 links, 183 joints
Links:
- link l_hand_index_1: geometry collision mesh filename=package://R1Mk3/meshes/simmechanics/sim_emorph_l_hand_index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 scale=0.001 0.001 0.001; visual mesh filename=package://R1Mk3/meshes/simmechanics/sim_emorph_l_hand_index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 scale=0.001 0.001 0.001
- link l_hand_index_2: geometry collision mesh filename=package://R1Mk3/meshes/simmechanics/sim_emorph_l_hand_index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 scale=0.001 0.001 0.001; visual mesh filename=package://R1Mk3/meshes/simmechanics/sim_emorph_l_hand_index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 scale=0.001 0.001 0.001
- link l_hand_index_3: geometry collision mesh filename=package://R1Mk3/meshes/simmechanics/sim_emorph_l_hand_index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 scale=0.001 0.001 0.001; visual mesh filename=package://R1Mk3/meshes/simmechanics/sim_emorph_l_hand_index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 scale=0.001 0.001 0.001
- link l_hand_middle_1: geometry collision mesh filename=package://R1Mk3/meshes/simmechanics/sim_emorph_l_hand_middl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 scale=0.001 0.001 0.001; visual mesh filename=package://R1Mk3/meshes/simmechanics/sim_emorph_l_hand_middl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 scale=0.001 0.001 0.001
- link l_hand_middle_2: geometry collision mesh filename=package://R1Mk3/meshes/simmechanics/sim_emorph_l_hand_middl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 scale=0.001 0.001 0.001; visual mesh filename=package://R1Mk3/meshes/simmechanics/sim_emorph_l_hand_middl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 scale=0.001 0.001 0.001
- link l_hand_palm: geometry collision mesh filename=package://R1Mk3/meshes/simmechanics/sim_emorph_l_hand_palm.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 scale=0.001 0.001 0.001; visual mesh filename=package://R1Mk3/meshes/simmechanics/sim_emorph_l_hand_palm.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 scale=0.001 0.001 0.001
- link l_hand_pinkie_1: geometry collision mesh filename=package://R1Mk3/meshes/simmechanics/sim_emorph_l_hand_pinki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 scale=0.001 0.001 0.001; visual mesh filename=package://R1Mk3/meshes/simmechanics/sim_emorph_l_hand_pinki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 scale=0.001 0.001 0.001
- link l_hand_pinkie_2: geometry collision mesh filename=package://R1Mk3/meshes/simmechanics/sim_emorph_l_hand_pinki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 scale=0.001 0.001 0.001; visual mesh filename=package://R1Mk3/meshes/simmechanics/sim_emorph_l_hand_pinki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 scale=0.001 0.001 0.001
- link l_hand_ring_1: geometry collision mesh filename=package://R1Mk3/meshes/simmechanics/sim_emorph_l_hand_ring_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 scale=0.001 0.001 0.001; visual mesh filename=package://R1Mk3/meshes/simmechanics/sim_emorph_l_hand_ring_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 scale=0.001 0.001 0.001
- link l_hand_ring_2: geometry collision mesh filename=package://R1Mk3/meshes/simmechanics/sim_emorph_l_hand_ring_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 scale=0.001 0.001 0.001; visual mesh filename=package://R1Mk3/meshes/simmechanics/sim_emorph_l_hand_ring_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 scale=0.001 0.001 0.001
- link l_hand_thumb_1: geometry collision mesh filename=package://R1Mk3/meshes/simmechanics/sim_emorph_l_hand_thumb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 scale=0.001 0.001 0.001; visual mesh filename=package://R1Mk3/meshes/simmechanics/sim_emorph_l_hand_thumb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 scale=0.001 0.001 0.001
- link l_hand_thumb_2: geometry collision mesh filename=package://R1Mk3/meshes/simmechanics/sim_emorph_l_hand_thumb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 scale=0.001 0.001 0.001; visual mesh filename=package://R1Mk3/meshes/simmechanics/sim_emorph_l_hand_thumb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 scale=0.001 0.001 0.001
- link l_hand_thumb_3: geometry collision mesh filename=package://R1Mk3/meshes/simmechanics/sim_emorph_l_hand_thumb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 scale=0.001 0.001 0.001; visual mesh filename=package://R1Mk3/meshes/simmechanics/sim_emorph_l_hand_thumb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 scale=0.001 0.001 0.001
- link r_hand_index_1: geometry collision mesh filename=package://R1Mk3/meshes/simmechanics/sim_emorph_r_hand_index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 scale=0.001 0.001 0.001; visual mesh filename=package://R1Mk3/meshes/simmechanics/sim_emorph_r_hand_index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 scale=0.001 0.001 0.001
- link r_hand_index_2: geometry collision mesh filename=package://R1Mk3/meshes/simmechanics/sim_emorph_r_hand_index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 scale=0.001 0.001 0.001; visual mesh filename=package://R1Mk3/meshes/simmechanics/sim_emorph_r_hand_index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 scale=0.001 0.001 0.001
- link r_hand_index_3: geometry collision mesh filename=package://R1Mk3/meshes/simmechanics/sim_emorph_r_hand_index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 scale=0.001 0.001 0.001; visual mesh filename=package://R1Mk3/meshes/simmechanics/sim_emorph_r_hand_index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 scale=0.001 0.001 0.001
- link r_hand_middle_1: geometry collision mesh filename=package://R1Mk3/meshes/simmechanics/sim_emorph_r_hand_middl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 scale=0.001 0.001 0.001; visual mesh filename=package://R1Mk3/meshes/simmechanics/sim_emorph_r_hand_middl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 scale=0.001 0.001 0.001
- link r_hand_middle_2: geometry collision mesh filename=package://R1Mk3/meshes/simmechanics/sim_emorph_r_hand_middl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 scale=0.001 0.001 0.001; visual mesh filename=package://R1Mk3/meshes/simmechanics/sim_emorph_r_hand_middl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 scale=0.001 0.001 0.001
- link r_hand_palm: geometry collision mesh filename=package://R1Mk3/meshes/simmechanics/sim_emorph_r_hand_palm.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 scale=0.001 0.001 0.001; visual mesh filename=package://R1Mk3/meshes/simmechanics/sim_emorph_r_hand_palm.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 scale=0.001 0.001 0.001
- link r_hand_pinkie_1: geometry collision mesh filename=package://R1Mk3/meshes/simmechanics/sim_emorph_r_hand_pinki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 scale=0.001 0.001 0.001; visual mesh filename=package://R1Mk3/meshes/simmechanics/sim_emorph_r_hand_pinki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 scale=0.001 0.001 0.001
- link r_hand_pinkie_2: geometry collision mesh filename=package://R1Mk3/meshes/simmechanics/sim_emorph_r_hand_pinki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 scale=0.001 0.001 0.001; visual mesh filename=package://R1Mk3/meshes/simmechanics/sim_emorph_r_hand_pinki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 scale=0.001 0.001 0.001
- link r_hand_ring_1: geometry collision mesh filename=package://R1Mk3/meshes/simmechanics/sim_emorph_r_hand_ring_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 scale=0.001 0.001 0.001; visual mesh filename=package://R1Mk3/meshes/simmechanics/sim_emorph_r_hand_ring_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 scale=0.001 0.001 0.001
- link r_hand_ring_2: geometry collision mesh filename=package://R1Mk3/meshes/simmechanics/sim_emorph_r_hand_ring_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 scale=0.001 0.001 0.001; visual mesh filename=package://R1Mk3/meshes/simmechanics/sim_emorph_r_hand_ring_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 scale=0.001 0.001 0.001
- link r_hand_thumb_1: geometry collision mesh filename=package://R1Mk3/meshes/simmechanics/sim_emorph_r_hand_thumb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 scale=0.001 0.001 0.001; visual mesh filename=package://R1Mk3/meshes/simmechanics/sim_emorph_r_hand_thumb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 scale=0.001 0.001 0.001
- link r_hand_thumb_2: geometry collision mesh filename=package://R1Mk3/meshes/simmechanics/sim_emorph_r_hand_thumb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 scale=0.001 0.001 0.001; visual mesh filename=package://R1Mk3/meshes/simmechanics/sim_emorph_r_hand_thumb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 scale=0.001 0.001 0.001
- link r_hand_thumb_3: geometry collision mesh filename=package://R1Mk3/meshes/simmechanics/sim_emorph_r_hand_thumb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 scale=0.001 0.001 0.001; visual mesh filename=package://R1Mk3/meshes/simmechanics/sim_emorph_r_hand_thumb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 scale=0.001 0.001 0.001
